Commit message: Update pvcchair.urdf.xacro
  <joint name="wheel_right_joint" type="continuous">
    <axis xyz="0 1 0" />
    <origin xyz="0 -0.02 0" rpy="0 0 0" />
    <parent link="wheel_axle_right" />
    <child link="wheel_right" />
  </joint>

  <joint name="wheel_left_joint" type="continuous">
    <axis xyz="0 1 0" />
    <origin xyz="0 +0.02 0" rpy="0 0 0" />
    <parent link="wheel_axle_left" />
    <child link="wheel_left" />
  </joint>

line 60

File: robot_ws/src/pvcchair_description/urdf/pvcchair.urdf.xacro (robot description, xacro)
@@ -38,15 +38,15 @@
     <child link="gearbox_plate_left" />
   </joint>
-  <joint name="wheel_right_joint" type="continuous">
-    <axis xyz="0 1 0" />
-    <origin xyz="0 -0.02 0" rpy="0 0 0" />
-    <parent link="wheel_axle_right" />
-    <child link="wheel_right" />
+    <joint name="swivel_right_joint2" type="continuous">
+    <axis xyz="0 0 1" />
+    <origin xyz="${-p1_hlen-2*c_offset-p3_len-c_offset+swivel_offset} ${-p2_hlen-c_offset} ${+c_offset+p9_len}" rpy="0 0 0" />
+    <parent link="base_link" />
+    <child link="swivel_right" />
   </joint>
-  <joint name="wheel_left_joint" type="continuous">
-    <axis xyz="0 1 0" />
-    <origin xyz="0 +0.02 0" rpy="0 0 0" />
-    <parent link="wheel_axle_left" />
-    <child link="wheel_left" />
+  <joint name="swivel_left_joint2" type="continuous">
+    <axis xyz="0 0 1" />
+    <origin xyz="${-p1_hlen-2*c_offset-p3_len-c_offset+swivel_offset} ${+p2_hlen+c_offset} ${+c_offset+p9_len}" rpy="0 0 0" />
+    <parent link="base_link" />
+    <child link="swivel_left" />
   </joint>
   <joint name="swivel_right_joint" type="continuous">

Commit message: Update pvcchair.urdf.xacro

File: robot_ws/src/pvcchair_description/urdf/pvcchair.urdf.xacro (robot description, xacro)
@@ -38,15 +38,15 @@
     <child link="gearbox_plate_left" />
   </joint>
-    <joint name="swivel_right_joint2" type="continuous">
-    <axis xyz="0 0 1" />
-    <origin xyz="${-p1_hlen-2*c_offset-p3_len-c_offset+swivel_offset} ${-p2_hlen-c_offset} ${+c_offset+p9_len}" rpy="0 0 0" />
-    <parent link="base_link" />
-    <child link="swivel_right" />
+<joint name="wheel_right_joint" type="continuous">
+  <axis xyz="0 1 0"/>
+  <origin xyz="0 -0.02 0" rpy="0 0 0"/>
+  <parent link="wheel_axle_right"/>
+  <child link="wheel_right"/>
   </joint>
-  <joint name="swivel_left_joint2" type="continuous">
-    <axis xyz="0 0 1" />
-    <origin xyz="${-p1_hlen-2*c_offset-p3_len-c_offset+swivel_offset} ${+p2_hlen+c_offset} ${+c_offset+p9_len}" rpy="0 0 0" />
-    <parent link="base_link" />
-    <child link="swivel_left" />
+  <joint name="wheel_left_joint" type="continuous">
+    <axis xyz="0 1 0"/>
+    <origin xyz="0 +0.02 0" rpy="0 0 0"/>
+    <parent link="wheel_axle_left"/>
+    <child link="wheel_left"/>
   </joint>
   <joint name="swivel_right_joint" type="continuous">
